File: Eagle/Beepoo.sch (EAGLE design)
At the start: 66 parts, among them CN1 JACK4PTH, CN2 SD-MICRO, CN3 USB-MC5F01, J1 JUMPER3-1.5MM, J2 JUMPER3-1.5MM, SW2 SLIDE1-PCM12, U1 RT9266-SOT23, U2 ATMEGA32U4, U3 AY-3-8912/28, U4 OPAMP-DUAL-SOIC8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

Commit message: Add reset to LCD. Connect A8 of AY to VCC
Connections:
- net +5V: now also U3.A8
- net AY_RESET: now also LCD1.!RST
- net GND: no longer U3.A8
Other:
- moved on the sheet: CN2, LCD1, R7
